File: hw/sch_pcb/SIPMPOWER01A/hw/sch_pcb/SIPMPOWER01A.kicad_pcb (KiCad board)
At the start: 2 copper layers, 60.5 x 40.1 mm, 33 parts, among them J1 HEADER_2x01_PARALLEL, J2 HEADER_2x01_PARALLEL, J3 HEADER_2x01_PARALLEL, J4 HEADER_2x01_PARALLEL, J5 HEADER_2x01_PARALLEL, M1 HOLE, M2 HOLE, M3 HOLE, M4 HOLE

Commit message: Edit
Parts:
- added J6: JUMP2_2x1, Mlab_Pin_Headers:Straight_1x02, F.Cu at (46.4, -11.4)
- R1, R3, R5, R7: value R -> 4k7
- R2, R4, R6, R8: value R -> 12k
- RV1, RV2, RV3, RV4: value 3296W -> 3296W-10k
- moved J1 0.63 mm to (47.6, -2.54)
- moved J2 0.63 mm to (47.6, -5.08)
Connections:
- C1 pad 1: Net-(BT1-Pad2) -> Net-(C1-Pad1)
- C2 pad 2: Net-(BT1-Pad2) -> Net-(C1-Pad1)
- C3 pad 2: Net-(BT1-Pad2) -> Net-(C1-Pad1)
- C4 pad 1: Net-(BT1-Pad2) -> Net-(C1-Pad1)
- C5 pad 1: Net-(BT1-Pad2) -> Net-(C1-Pad1)
Routing:
- net Net-(C1-Pad3): track 0.00 -> 23.9 mm, vias 0 -> 2
- net Net-(C1-Pad1): track 0.00 -> 22.0 mm
- net /U2: track 2.43 -> 17.8 mm
- net /U3: track 5.87 -> 20.6 mm
- net Net-(BT3-Pad1): track 56.3 -> 65.8 mm
- net Net-(BT1-Pad2): track 13.4 -> 5.15 mm
- net /U1: track 14.0 -> 16.5 mm
- net Net-(R6-Pad1): track 0.00 -> 2.43 mm
- net /U4: track 15.9 -> 15.4 mm
- added copper zone on B.Cu, net GND
- added copper zone on F.Cu, net GND
Other:
- board text added: "SIPMPOWER01A"
- board text removed: "CAT."
- board text removed: "GND"
- board text removed: "SIPM01A"

Commit message: Modifications
Parts:
- added J7: HEADER_2x01, Mlab_Pin_Headers:Straight_1x02, F.Cu at (2.03, -29.7)
- added J8: HEADER_2x01, Mlab_Pin_Headers:Straight_1x02, F.Cu at (4.57, -29.7)
- added J9: HEADER_2x01, Mlab_Pin_Headers:Straight_1x02, F.Cu at (7.11, -29.7)
Connections:
- net Net-(BT1-Pad2) renamed /-
- net Net-(BT3-Pad1) renamed /+
Routing:
- net /-: track 5.15 -> 50.5 mm
- net /+: track 65.8 -> 108.3 mm, vias 0 -> 1
- net Net-(J8-Pad2): track 0.00 -> 3.59 mm
- net Net-(J7-Pad2): track 0.00 -> 3.59 mm
