File: hw/sch_pcb/SIPMPOWER01A/hw/sch_pcb/SIPMPOWER01A.sch (KiCad schematic (older format))
At the start: 33 parts, among them J1 HEADER_2x01_PARALLEL, J2 HEADER_2x01_PARALLEL, J3 HEADER_2x01_PARALLEL, J4 HEADER_2x01_PARALLEL, J5 HEADER_2x01_PARALLEL, M1 HOLE, M2 HOLE, M3 HOLE, M4 HOLE

Commit message: Edit
Parts:
- added J6: JUMP2_2x1, Mlab_Pin_Headers:Straight_1x02, symbol MLAB_Jumpers:JUMP2_2x1
- R1, R3, R5, R7: value R -> 4k7
- R2, R4, R6, R8: value R -> 12k
- RV1, RV2, RV3, RV4: value 3296W -> 3296W-10k
Connections:
- net at C1.1, C2.2, C3.2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: now also J6.1; no longer BT1.2 (-)
- new net: BT1.2 (-), J6.2 (1)
Other:
- moved on the sheet: C1, C2, C3, C4, C5, C6, C7, C8, C9, J1, J2, J3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

Commit message: Modifications
Parts:
- added J7, J8, J9: HEADER_2x01, Mlab_Pin_Headers:Straight_1x02, symbol MLAB_HEADER:HEADER_2x01
Connections:
- net -: now reaches BT1.2 (-), J6.2 (1)
- net -: now also J9.2
- net +: now reaches BT3.1 (+), C1.2, C2.1, C3.1, C4.2, C5.2, C6.2, C7.2, C8.2, C9.2, J5.1, J5.2, R2.2, R4.2, R6.2, R8.2
- net +: now also J7.1
- new net: J7.2, J8.1
- new net: J8.2, J9.1
Changed lines of the file:
@@
 	2200 2900 2650 2900
 Connection ~ 2650 2900
+$Comp
+L MLAB_HEADER:HEADER_2x01 J7
+U 1 1 5BB16337
+P 2660 1290
+F 0 "J7" H 2660 1431 60  0000 C CNN
+F 1 "HEADER_2x01" H 2660 1431 60  0001 C CNN
+F 2 "Mlab_Pin_Headers:Straight_1x02" H 2660 1290 60  0001 C CNN
+F 3 "" H 2660 1290 60  0000 C CNN
+	1    2660 1290
+	1    0    0    -1
+$EndComp
+$Comp
+L MLAB_HEADER:HEADER_2x01 J8
+U 1 1 5BB165B3
+P 2660 1600
+F 0 "J8" H 2660 1741 60  0000 C CNN
+F 1 "HEADER_2x01" H 2660 1741 60  0001 C CNN
+F 2 "Mlab_Pin_Headers:Straight_1x02" H 2660 1600 60  0001 C CNN
+F 3 "" H 2660 1600 60  0000 C CNN
+	1    2660 1600
+	1    0    0    -1
+$EndComp
+$Comp
+L MLAB_HEADER:HEADER_2x01 J9
+U 1 1 5BB16655
+P 2660 1940
+F 0 "J9" H 2660 2081 60  0000 C CNN
+F 1 "HEADER_2x01" H 2660 2081 60  0001 C CNN
+F 2 "Mlab_Pin_Headers:Straight_1x02" H 2660 1940 60  0001 C CNN
+F 3 "" H 2660 1940 60  0000 C CNN
+	1    2660 1940
+	1    0    0    -1
+$EndComp
+Wire Wire Line
+	2410 1600 2410 1380
+Wire Wire Line
+	2410 1380 2910 1380
+Wire Wire Line
+	2910 1380 2910 1290
+Wire Wire Line
+	2910 1600 2910 1700
+Wire Wire Line
+	2910 1700 2410 1700
+Wire Wire Line
+	2410 1700 2410 1940
+Wire Wire Line
+	2410 1290 2350 1290
+Wire Wire Line
+	2910 1940 2930 1940
+Text Label 2350 1290 0    60   ~ 0
++
+Text Label 2930 1940 0    60   ~ 0
+-
+Text Label 1100 2900 0    60   ~ 0
+-
+Text Label 1100 4000 0    60   ~ 0
++
 $EndSCHEMATC
