File: hw/sch_pcb/SIPM01A/hw/sch_pcb/SIPM01A.kicad_pcb (KiCad board)
At the start: 2 copper layers, 19.8 x 40.1 mm, 20 parts, among them J1 HEADER_1x01, J2 HEADER_1x01, J3 HEADER_1x01, J4 HEADER_1x01, J5 CONN_2, J6 CONN_2, J7 HEADER_1x01, M1 HOLE, M2 HOLE, M3 HOLE, M4 HOLE, U1 ARRAYC-60035-4P-BGA

Commit message: Edit
Other:
- board text removed: "JACHO"
Changed lines of the file:
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@@
   (page A4)
   (layers
-    (0 F.Cu signal)
-    (31 B.Cu signal)
+    (0 F.Cu signal hide)
+    (31 B.Cu signal hide)
     (32 B.Adhes user)
     (33 F.Adhes user)
@@
   )
   (setup
-    (last_trace_width 0.8)
+    (last_trace_width 0.25)
     (user_trace_width 0.4)
     (user_trace_width 0.5)
@@
       (effects (font (size 1 1) (thickness 0.15)))
     )
-    (fp_text value ARRAYC-60035-4P-BGA (at 0.1524 2.5146) (layer F.Fab)
+    (fp_text value ARRAYC-60035-4P-BGA (at 0.1524 2.5146) (layer F.Fab) hide
       (effects (font (size 1 1) (thickness 0.15)))
     )
@@
     (tags "capacitor handsolder")
     (attr smd)
-    (fp_text reference C1 (at 0 1.85 90) (layer B.SilkS)
-      (effects (font (size 1 1) (thickness 0.15)) (justify mirror))
-    )
-    (fp_text value EMI_Filter_C (at 0 -1.85 90) (layer B.Fab)
+    (fp_text reference C1 (at 0 0 90) (layer B.SilkS)
+      (effects (font (size 1 1) (thickness 0.15)) (justify mirror))
+    )
+    (fp_text value EMI_Filter_C (at 0 -1.85 90) (layer B.Fab) hide
       (effects (font (size 1 1) (thickness 0.15)) (justify mirror))
     )
@@
     (tags "Tantal Cap. , Size C, EIA-6032, Reflow,")
     (attr smd)
-    (fp_text reference C2 (at 0 2.85 180) (layer B.SilkS)
+    (fp_text reference C2 (at 0.01524 0 180) (layer B.SilkS)
       (effects (font (size 1.524 1.524) (thickness 0.3048)) (justify mirror))
     )
@@
     (tags "capacitor handsolder")
     (attr smd)
-    (fp_text reference C4 (at 0 1.85) (layer B.SilkS)
-      (effects (font (size 1 1) (thickness 0.15)) (justify mirror))
-    )
-    (fp_text value EMI_Filter_C (at 0 -1.85) (layer B.Fab)
+    (fp_text reference C4 (at 0.1825 0) (layer B.SilkS)
+      (effects (font (size 1 1) (thickness 0.15)) (justify mirror))
+    )
+    (fp_text value EMI_Filter_C (at 0 -1.85) (layer B.Fab) hide
       (effects (font (size 1 1) (thickness 0.15)) (justify mirror))
     )
@@
     (tags "Tantal Cap. , Size C, EIA-6032, Reflow,")
     (attr smd)
-    (fp_text reference C5 (at 0 2.85 90) (layer B.SilkS)
+    (fp_text reference C5 (at 0.01524 0 90) (layer B.SilkS)
       (effects (font (size 1.524 1.524) (thickness 0.3048)) (justify mirror))
     )
@@
     (tags "capacitor handsolder")
     (attr smd)
-    (fp_text reference C7 (at 0 1.85 90) (layer B.SilkS)
-      (effects (font (size 1 1) (thickness 0.15)) (justify mirror))
-    )
-    (fp_text value EMI_Filter_C (at 0 -1.85 90) (layer B.Fab)
+    (fp_text reference C7 (at 0 0 90) (layer B.SilkS)
+      (effects (font (size 1 1) (thickness 0.15)) (justify mirror))
+    )
+    (fp_text value EMI_Filter_C (at 0 -1.85 90) (layer B.Fab) hide
       (effects (font (size 1 1) (thickness 0.15)) (justify mirror))
     )
@@
     (tags "capacitor handsolder")
     (attr smd)
-    (fp_text reference C10 (at 0 1.85 90) (layer B.SilkS)
-      (effects (font (size 1 1) (thickness 0.15)) (justify mirror))
-    )
-    (fp_text value EMI_Filter_C (at 0 -1.85 90) (layer B.Fab)
+    (fp_text reference C10 (at 0 0 90) (layer B.SilkS)
+      (effects (font (size 1 1) (thickness 0.15)) (justify mirror))
+    )
+    (fp_text value EMI_Filter_C (at 0 -1.85 90) (layer B.Fab) hide
       (effects (font (size 1 1) (thickness 0.15)) (justify mirror))
     )
@@
     (tags "Tantal Cap. , Size C, EIA-6032, Reflow,")
     (attr smd)
-    (fp_text reference C3 (at 0 2.85) (layer B.SilkS)
+    (fp_text reference C3 (at 0.01524 0) (layer B.SilkS)
       (effects (font (size 1.524 1.524) (thickness 0.3048)) (justify mirror))
     )
@@
     (tags "Tantal Cap. , Size C, EIA-6032, Reflow,")
     (attr smd)
-    (fp_text reference C6 (at 0 2.85 90) (layer B.SilkS)
+    (fp_text reference C6 (at -0.01524 0 90) (layer B.SilkS)
       (effects (font (size 1.524 1.524) (thickness 0.3048)) (justify mirror))
     )
@@
     (effects (font (size 1.5 1.5) (thickness 0.3)) (justify mirror))
   )
-  (gr_text 2018 (at -24.765 -8.89) (layer F.SilkS)
+  (gr_text 2018 (at 10.16 -5.08 90) (layer F.SilkS)
     (effects (font (size 1.5 1.5) (thickness 0.3)))
   )
-  (gr_text JACHO (at -26.67 -15.875) (layer F.SilkS)
+  (gr_text SIPM01A (at 10.16 -34.29 90) (layer F.SilkS)
     (effects (font (size 1.5 1.5) (thickness 0.3)))
   )

Commit message: Modifications
Other:
- board text removed: "MLAB.CZ"
- board text removed: "U2"
- board text removed: "U3"
- board text removed: "U4"
Changed lines of the file:
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@@
-(kicad_pcb (version 20171130) (host pcbnew "(2018-02-10 revision a04965c36)-makepkg")
+(kicad_pcb (version 20171130) (host pcbnew 6.0.0-rc1-unknown-f68581d~66~ubuntu16.04.1)
   (general
     (thickness 1.6)
-    (drawings 14)
+    (drawings 8)
     (tracks 66)
     (zones 0)
@@
   (page A4)
   (layers
-    (0 F.Cu signal hide)
-    (31 B.Cu signal hide)
+    (0 F.Cu signal)
+    (31 B.Cu signal)
     (32 B.Adhes user)
     (33 F.Adhes user)
@@
     (zone_45_only no)
     (trace_min 0.2)
-    (segment_width 0.2)
-    (edge_width 0.15)
     (via_size 0.8)
     (via_drill 0.4)
@@
     (uvia_min_size 0.2)
     (uvia_min_drill 0.1)
+    (edge_width 0.15)
+    (segment_width 0.2)
     (pcb_text_width 0.3)
     (pcb_text_size 1.5 1.5)
@@
     (pad_drill 0)
     (pad_to_mask_clearance 0.2)
+    (solder_mask_min_width 0.25)
     (aux_axis_origin 0 0)
     (visible_elements 7FFFFF7F)
     (pcbplotparams
-      (layerselection 0x010fc_ffffffff)
+      (layerselection 0x010e0_ffffffff)
       (usegerberextensions false)
       (usegerberattributes false)
@@
       (hpglpennumber 1)
       (hpglpenspeed 20)
-      (hpglpendiameter 15)
+      (hpglpendiameter 15.000000)
       (psnegative false)
       (psa4output false)
@@
       (outputformat 1)
       (mirror false)
-      (drillshape 1)
+      (drillshape 0)
       (scaleselection 1)
-      (outputdirectory ""))
+      (outputdirectory "CAM_PROFI/"))
   )
   (net 0 "")
@@
     (pad 2 smd trapezoid (at 0 0 90) (size 1.5 3) (layers B.Cu B.Paste B.Mask)
       (net 11 /+))
-    (pad 3 smd roundrect (at 2.0875 0 90) (size 1.575 1.8) (layers B.Cu B.Paste B.Mask)(roundrect_rratio 0.159)
+    (pad 3 smd roundrect (at 2.0875 0 90) (size 1.575 1.8) (layers B.Cu B.Paste B.Mask) (roundrect_rratio 0.159)
       (net 1 /U1))
-    (pad 1 smd roundrect (at -2.0875 0 90) (size 1.575 1.8) (layers B.Cu B.Paste B.Mask)(roundrect_rratio 0.15873)
+    (pad 1 smd roundrect (at -2.0875 0 90) (size 1.575 1.8) (layers B.Cu B.Paste B.Mask) (roundrect_rratio 0.15873)
       (net 6 /U1in))
     (model ${KISYS3DMOD}/Capacitor_SMD.3dshapes/C_1806_4516Metric.wrl
@@
       (effects (font (size 1 1) (thickness 0.15)) (justify mirror))
     )
-    (pad 1 smd roundrect (at -2.0875 0) (size 1.575 1.8) (layers B.Cu B.Paste B.Mask)(roundrect_rratio 0.15873)
+    (pad 1 smd roundrect (at -2.0875 0) (size 1.575 1.8) (layers B.Cu B.Paste B.Mask) (roundrect_rratio 0.15873)
       (net 7 /U2in))
-    (pad 3 smd roundrect (at 2.0875 0) (size 1.575 1.8) (layers B.Cu B.Paste B.Mask)(roundrect_rratio 0.159)
+    (pad 3 smd roundrect (at 2.0875 0) (size 1.575 1.8) (layers B.Cu B.Paste B.Mask) (roundrect_rratio 0.159)
       (net 2 /U2))
     (pad 2 smd trapezoid (at 0 0) (size 1.5 3) (layers B.Cu B.Paste B.Mask)
@@
     (pad 2 smd trapezoid (at 0 0 90) (size 1.5 3) (layers B.Cu B.Paste B.Mask)
       (net 11 /+))
-    (pad 3 smd roundrect (at 2.0875 0 90) (size 1.575 1.8) (layers B.Cu B.Paste B.Mask)(roundrect_rratio 0.159)
+    (pad 3 smd roundrect (at 2.0875 0 90) (size 1.575 1.8) (layers B.Cu B.Paste B.Mask) (roundrect_rratio 0.159)
       (net 3 /U3))
-    (pad 1 smd roundrect (at -2.0875 0 90) (size 1.575 1.8) (layers B.Cu B.Paste B.Mask)(roundrect_rratio 0.15873)
+    (pad 1 smd roundrect (at -2.0875 0 90) (size 1.575 1.8) (layers B.Cu B.Paste B.Mask) (roundrect_rratio 0.15873)
       (net 8 /U3in))
     (model ${KISYS3DMOD}/Capacitor_SMD.3dshapes/C_1806_4516Metric.wrl
@@
       (effects (font (size 1 1) (thickness 0.15)) (justify mirror))
     )
-    (pad 1 smd roundrect (at -2.0875 0 90) (size 1.575 1.8) (layers B.Cu B.Paste B.Mask)(roundrect_rratio 0.15873)
+    (pad 1 smd roundrect (at -2.0875 0 90) (size 1.575 1.8) (layers B.Cu B.Paste B.Mask) (roundrect_rratio 0.15873)
       (net 9 /U4in))
-    (pad 3 smd roundrect (at 2.0875 0 90) (size 1.575 1.8) (layers B.Cu B.Paste B.Mask)(roundrect_rratio 0.159)
+    (pad 3 smd roundrect (at 2.0875 0 90) (size 1.575 1.8) (layers B.Cu B.Paste B.Mask) (roundrect_rratio 0.159)
       (net 4 /U4))
     (pad 2 smd trapezoid (at 0 0 90) (size 1.5 3) (layers B.Cu B.Paste B.Mask)
@@
     (effects (font (size 1.5 1.5) (thickness 0.3)) (justify left))
   )
-  (gr_text U4 (at 142.875 -27.305) (layer F.SilkS)
-    (effects (font (size 1.5 1.5) (thickness 0.3)) (justify left))
-  )
-  (gr_text U3 (at 142.875 -29.845) (layer F.SilkS)
-    (effects (font (size 1.5 1.5) (thickness 0.3)) (justify left))
-  )
-  (gr_text U2 (at 142.875 -32.385) (layer F.SilkS)
-    (effects (font (size 1.5 1.5) (thickness 0.3)) (justify left))
-  )
   (gr_text + (at 16.51 -11.43) (layer F.SilkS)
     (effects (font (size 1.5 1.5) (thickness 0.3)) (justify left))
   )
-  (gr_text MLAB.CZ (at -27.305 -19.685) (layer B.Cu)
-    (effects (font (size 1.5 1.5) (thickness 0.3)) (justify mirror))
-  )
   (gr_text 2018 (at 10.16 -5.08 90) (layer F.SilkS)
     (effects (font (size 1.5 1.5) (thickness 0.3)))
   )
   (gr_text SIPM01A (at 10.16 -34.29 90) (layer F.SilkS)
-    (effects (font (size 1.5 1.5) (thickness 0.3)))
-  )
-  (gr_text SIPM01A (at 140.97 -20.32) (layer F.SilkS)
-    (effects (font (size 1.5 1.5) (thickness 0.3)))
-  )
-  (gr_text MLAB.CZ (at 140.97 -22.86) (layer F.SilkS)
     (effects (font (size 1.5 1.5) (thickness 0.3)))
   )
@@
   (segment (start 9.795 -22.86) (end 6.35 -22.86) (width 0.8) (layer B.Cu) (net 7))
   (via (at 6.35 -22.86) (size 0.8) (drill 0.4) (layers F.Cu B.Cu) (net 7))
+  (segment (start 9.525 -11.43) (end 9.525 -14.4225) (width 0.8) (layer B.Cu) (net 8) (status 30))
+  (segment (start 9.525 -14.4225) (end 10.16 -15.0575) (width 0.8) (layer B.Cu) (net 8) (status 30))
+  (segment (start 12.065 -11.43) (end 12.065 -13.1525) (width 0.8) (layer B.Cu) (net 9) (status 10))
+  (segment (start 12.065 -13.1525) (end 13.97 -15.0575) (width 0.8) (layer B.Cu) (net 9) (status 20))
   (segment (start 18.0032 -30.6397) (end 18.034 -30.6705) (width 0.25) (layer F.Cu) (net 10))
   (segment (start 18.0032 -25.293) (end 18.0032 -30.6397) (width 0.25) (layer F.Cu) (net 10))
@@
   (segment (start 17.78 -13.98524) (end 14.62024 -17.145) (width 0.8) (layer B.Cu) (net 11) (status 20))
   (segment (start 14.62024 -17.145) (end 13.97 -17.145) (width 0.8) (layer B.Cu) (net 11) (status 30))
-  (segment (start 9.525 -11.43) (end 9.525 -14.4225) (width 0.8) (layer B.Cu) (net 8) (status 30))
-  (segment (start 9.525 -14.4225) (end 10.16 -15.0575) (width 0.8) (layer B.Cu) (net 8) (status 30))
-  (segment (start 12.065 -11.43) (end 12.065 -13.1525) (width 0.8) (layer B.Cu) (net 9) (status 10))
-  (segment (start 12.065 -13.1525) (end 13.97 -15.0575) (width 0.8) (layer B.Cu) (net 9) (status 20))
   (zone (net 5) (net_name GND) (layer F.Cu) (hatch edge 0.508)
     (connect_pads yes (clearance 0.508))

Commit message: Edit
Parts:
- C1, C10, C4, C7: value EMI_Filter_C -> 1u5/50V - NFM41PC155B1H3L
Changed lines of the file:
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@@
-(kicad_pcb (version 20171130) (host pcbnew 6.0.0-rc1-unknown-f68581d~66~ubuntu16.04.1)
+(kicad_pcb (version 20171130) (host pcbnew "(6.0.0-rc1-dev-205-gc0615c5ef)")
   (general
     (thickness 1.6)
@@
       (effects (font (size 1 1) (thickness 0.15)) (justify mirror))
     )
-    (fp_text value EMI_Filter_C (at 0 -1.85 90) (layer B.Fab) hide
+    (fp_text value "1u5/50V - NFM41PC155B1H3L" (at 0 -1.85 90) (layer B.Fab) hide
       (effects (font (size 1 1) (thickness 0.15)) (justify mirror))
     )
@@
       (effects (font (size 1 1) (thickness 0.15)) (justify mirror))
     )
-    (fp_text value EMI_Filter_C (at 0 -1.85) (layer B.Fab) hide
+    (fp_text value "1u5/50V - NFM41PC155B1H3L" (at 0 -1.85) (layer B.Fab) hide
       (effects (font (size 1 1) (thickness 0.15)) (justify mirror))
     )
@@
       (effects (font (size 1 1) (thickness 0.15)) (justify mirror))
     )
-    (fp_text value EMI_Filter_C (at 0 -1.85 90) (layer B.Fab) hide
+    (fp_text value "1u5/50V - NFM41PC155B1H3L" (at 0 -1.85 90) (layer B.Fab) hide
       (effects (font (size 1 1) (thickness 0.15)) (justify mirror))
     )
@@
       (effects (font (size 1 1) (thickness 0.15)) (justify mirror))
     )
-    (fp_text value EMI_Filter_C (at 0 -1.85 90) (layer B.Fab) hide
-      (effects (font (size 1 1) (thickness 0.15)) (justify mirror))
-    )
+    (fp_text value "1u5/50V - NFM41PC155B1H3L" (at 0 -1.85 90) (layer B.Fab) hide
+      (effects (font (size 1 1) (thickness 0.15)) (justify mirror))
+    )
