File: hw/sch_pcb/SIPM01A/hw/sch_pcb/SIPM01A.sch (KiCad schematic (older format))
At the start: 20 parts, among them J1 HEADER_1x01, J2 HEADER_1x01, J3 HEADER_1x01, J4 HEADER_1x01, J5 CONN_2, J6 CONN_2, J7 HEADER_1x01, M1 HOLE, M2 HOLE, M3 HOLE, M4 HOLE, U1 ARRAYC-60035-4P-BGA

Commit message: Edit
Parts:
- C1, C10, C4, C7: value EMI_Filter_C -> 1u5/50V - NFM41PC155B1H3L
Changed lines of the file:
@@
 P 3050 3500
 F 0 "C1" H 3050 3805 50  0000 C CNN
-F 1 "EMI_Filter_C" H 3050 3714 50  0000 C CNN
+F 1 "1u5/50V - NFM41PC155B1H3L" H 3050 3714 50  0000 C CNN
 F 2 "Mlab_L:FIR_1806" V 3050 3500 50  0001 C CNN
 F 3 "http://www.murata.com/~/media/webrenewal/support/library/catalog/products/emc/emifil/c31e.ashx?la=en-gb" V 3050 3500 50  0001 C CNN
@@
 P 7100 3500
 F 0 "C10" H 7100 3805 50  0000 C CNN
-F 1 "EMI_Filter_C" H 7100 3714 50  0000 C CNN
+F 1 "1u5/50V - NFM41PC155B1H3L" H 7100 3714 50  0000 C CNN
 F 2 "Mlab_L:FIR_1806" V 7100 3500 50  0001 C CNN
 F 3 "http://www.murata.com/~/media/webrenewal/support/library/catalog/products/emc/emifil/c31e.ashx?la=en-gb" V 7100 3500 50  0001 C CNN
@@
 P 5750 3500
 F 0 "C7" H 5750 3805 50  0000 C CNN
-F 1 "EMI_Filter_C" H 5750 3714 50  0000 C CNN
+F 1 "1u5/50V - NFM41PC155B1H3L" H 5750 3714 50  0000 C CNN
 F 2 "Mlab_L:FIR_1806" V 5750 3500 50  0001 C CNN
 F 3 "http://www.murata.com/~/media/webrenewal/support/library/catalog/products/emc/emifil/c31e.ashx?la=en-gb" V 5750 3500 50  0001 C CNN
@@
 P 4400 3500
 F 0 "C4" H 4400 3805 50  0000 C CNN
-F 1 "EMI_Filter_C" H 4400 3714 50  0000 C CNN
+F 1 "1u5/50V - NFM41PC155B1H3L" H 4400 3714 50  0000 C CNN
 F 2 "Mlab_L:FIR_1806" V 4400 3500 50  0001 C CNN
 F 3 "http://www.murata.com/~/media/webrenewal/support/library/catalog/products/emc/emifil/c31e.ashx?la=en-gb" V 4400 3500 50  0001 C CNN
