File: hw/sch_pcb/AIRDOSC01A_PCB01A/hw/sch_pcb/AIRDOSC01A_PCB01A.kicad_pcb (KiCad board)
At the start: 2 copper layers, 2 parts, among them U2 MICROFC-60035-SMT-TR(1), U3 MICROFC-60035-SMT-TR(1)

Commit message: edit
Parts:
- removed U3: MICROFC-60035-SMT-TR(1), Mlab_IO:MicroFC−60035−SMT
- added C1: 15uF/35V, Mlab_C:TantalC_SizeC_Reflow, F.Cu at (37.2, 33.8)
- added C10: -, Mlab_R:SMD-0805, F.Cu at (61.7, 44.1)
- added C2: 1u5/50V - NFM41PC155B1H3L, Mlab_L:FIR_1806, F.Cu at (50.5, 39.4)
- added C3: 47uF, Mlab_C:TantalC_SizeC_Reflow, F.Cu at (37.2, 38.7)
- added C4: 10u, Mlab_R:SMD-0805, F.Cu at (61.7, 42.3)
- added C5: 100nF, Mlab_R:SMD-0805, F.Cu at (61.7, 40.5)
- added C6: 10nF, Mlab_R:SMD-0805, F.Cu at (58.3, 44.2)
- added C7: 10u, Mlab_R:SMD-0805, F.Cu at (64.2, 38.7)
- added C8: 100nF, Mlab_R:SMD-0805, F.Cu at (60.7, 36.9)
- added C9: 10nF, Mlab_R:SMD-0805, F.Cu at (54.8, 47.1)
- added D1: M4, Mlab_D:Diode-SMA_Standard, F.Cu at (35.0, 42.3)
- added J1: HEADER_2x01_PARALLEL, Mlab_Pin_Headers:Straight_2x01, F.Cu at (62.3, 32.0)
- added J2: HEADER_2x01_PARALLEL, Mlab_Pin_Headers:Straight_2x01, F.Cu at (46.9, 48.3)
- added J3: HEADER_2x01_PARALLEL, Mlab_Pin_Headers:Straight_2x01, F.Cu at (56.3, 38.4)
- added J4: HEADER_2x01_PARALLEL, Mlab_Pin_Headers:Straight_2x01, F.Cu at (46.9, 45.6)
- added J5: HEADER_2x01_PARALLEL, Mlab_Pin_Headers:Straight_2x01, F.Cu at (50.0, 42.2)
- added J6: HEADER_2x01_PARALLEL, Mlab_Pin_Headers:Straight_2x01, F.Cu at (57.1, 34.7)
- added J7: HEADER_2x01_PARALLEL, Mlab_Pin_Headers:Straight_2x01, F.Cu at (57.1, 32.0)
- added J8: HEADER_2x01_PARALLEL, Mlab_Pin_Headers:Straight_2x01, F.Cu at (62.3, 34.7)
- added M1: HOLE, Mlab_Mechanical:MountingHole_3mm, F.Cu at (34.7, 47.2)
- added M2: HOLE, Mlab_Mechanical:MountingHole_3mm, F.Cu at (44.2, 41.0)
- added M3: HOLE, Mlab_Mechanical:MountingHole_3mm, F.Cu at (51.3, 33.9)
- added M4: HOLE, Mlab_Mechanical:MountingHole_3mm, F.Cu at (41.1, 47.4)
- added R1: 1k, Mlab_R:SMD-0805, F.Cu at (51.3, 47.1)
- added R10: 1k, Mlab_R:SMD-0805, F.Cu at (58.2, 47.8)
- added R11: 0R, Mlab_R:SMD-0805, F.Cu at (65.2, 40.5)
- added R12: 1k, Mlab_R:SMD-0805, F.Cu at (54.8, 48.9)
- added R2: 10R, Mlab_R:SMD-0805, F.Cu at (51.3, 48.9)
- added R3: 100R, Mlab_R:SMD-0805, F.Cu at (54.8, 45.3)
- added R4: 10R, Mlab_R:SMD-0805, F.Cu at (60.7, 38.7)
- added R5: 0R, Mlab_R:SMD-0805, F.Cu at (58.3, 40.6)
- added R6: 0R, Mlab_R:SMD-0805, F.Cu at (51.3, 45.3)
- added R7: 2k, Mlab_R:SMD-0805, F.Cu at (58.3, 42.4)
- added R8: 2k, Mlab_R:SMD-0805, F.Cu at (64.2, 36.9)
- added R9: 1k, Mlab_R:SMD-0805, F.Cu at (58.2, 46.0)
- added U1: MICROFC-60035-SMT-TR(1), Mlab_IO:MicroFC−60035−SMT, F.Cu at (44.5, 34.3)
- U2: value MICROFC-60035-SMT-TR(1) -> OPA836IDB; footprint Mlab_IO:MicroFC−60035−SMT -> Package_TO_SOT_SMD:SOT-23-6
- moved U2 203.3 mm to (37.8, 22.7)
Connections:
- U2 pad 1: /A -> Net-(R10-Pad1)
- U2 pad 2: (no net) -> GND
- U2 pad 3: /K -> /DIRECT_OUT
- U2 pad 4: (no net) -> Net-(R10-Pad2)
- U2 pad 5: (no net) -> /#PD
- U2 pad 6: (no net) -> +3V3

Commit message: edit
Parts:
- removed the J7 at (57.1, 32.0)
- added J10: HEADER_2x01_PARALLEL, Mlab_Pin_Headers:Straight_2x01, F.Cu at (26.4, -20.8)
- added J4: HEADER_2x01_PARALLEL, Mlab_Pin_Headers:Straight_2x01, F.Cu at (26.4, -2.54)
- added J9: HEADER_2x01_PARALLEL, Mlab_Pin_Headers:Straight_2x01, F.Cu at (26.4, -15.7)
- C1, C10, C2, C3, C4, C5, C6, C7, C8, C9, D1, R1, R10, R11, R12, R2, R3, R4, R5, R6, R7, R8, R9, U2: moved to B.Cu
- moved M4 86.9 mm to (15.2, -35.6)
- moved R1 86.9 mm to (21.8, -34.6), turned to 90 degrees
- moved C6 86.6 mm to (9.59, -27.4), turned to 180 degrees
- moved J2 86.3 mm to (26.4, -35.6)
- moved R4 85.7 mm to (10.2, -30.5)
- moved C5 85.4 mm to (14.3, -30.5)
- moved R2 84.9 mm to (14.2, -27.4)
- moved C9 84.5 mm to (10.6, -24.9), turned to 180 degrees
- moved M3 83.4 mm to (5.08, -35.6)
- moved J3 82.1 mm to (26.4, -38.1)
- moved R10 79.6 mm to (18.7, -21.3)
- moved C10 78.9 mm to (9.72, -15.2), turned to 180 degrees
- moved R9 77.4 mm to (21.8, -22.3), turned to 90 degrees
- moved R6 75.5 mm to (13.2, -19.9), turned to 90 degrees
- moved R5 75.0 mm to (6.60, -13.8), turned to 90 degrees
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- renumbered J4 to J5, J5 to J6, J6 to J7
Connections:
- J8 pad 1: /#PD -> /OUT
- J8 pad 2: /#PD -> /OUT
Routing:
- net GND: track 0.00 -> 51.0 mm, vias 0 -> 44
- net /DIRECT_OUT: track 0.00 -> 27.0 mm, vias 0 -> 1
- net /+3V6: track 0.00 -> 17.7 mm
- net +3V3: track 0.00 -> 15.4 mm
- net /OUT: track 0.00 -> 13.0 mm, vias 0 -> 1
- net /#PD: track 0.00 -> 10.4 mm
- net Net-(C6-Pad1): track 0.00 -> 9.38 mm, vias 0 -> 1
- net Net-(C1-Pad1): track 0.00 -> 8.33 mm
- net Net-(R10-Pad1): track 0.00 -> 8.02 mm, vias 0 -> 2
- net +28V: track 0.00 -> 5.84 mm
- net Net-(C5-Pad1): track 0.00 -> 5.23 mm
- net Net-(R10-Pad2): track 0.00 -> 4.77 mm
- net Net-(C10-Pad2): track 0.00 -> 4.49 mm, vias 0 -> 1
- net Net-(C2-Pad3): track 0.00 -> 3.69 mm
- net Net-(R6-Pad1): track 0.00 -> 2.68 mm, vias 0 -> 1
- added copper zone on B.Cu, net GND
- added copper zone on F.Cu, net GND
Other:
- board outline added: 30 x 40.1 mm
- board text added: "#PD"
- board text added: "DIROUT"
- board text added: "GND"
- board text added: "IN 28V"
- board text added: "IN 3V6"
- board text added: "OUT"
- board text added: "UST.CZ AIRDOSC01A_PCB01A"
