File: hw/sch_pcb/AIRDOSC01A_PCB01A/hw/sch_pcb/AIRDOSC01A_PCB01A.sch (KiCad schematic (older format))
At the start: 20 parts, among them J1 HEADER_1x01, J2 HEADER_1x01, J3 HEADER_1x01, J4 HEADER_1x01, J5 CONN_2, J6 CONN_2, J7 HEADER_1x01, M1 HOLE, M2 HOLE, M3 HOLE, M4 HOLE, U1 ARRAYC-60035-4P-BGA

Commit message: edit
Parts:
- added U2, U3: MICROFC-60035-SMT-TR(1), Mlab_IO:MicroFC−60035−SMT, symbol MLAB_IO:MICROFC-60035-SMT-TR(1)
Connections:
- net labels added: A
- wire segments 55 -> 61
Changed lines of the file:
@@
 EESchema Schematic File Version 4
-LIBS:SIPM01A-cache
-EELAYER 26 0
+EELAYER 29 0
 EELAYER END
 $Descr A4 11693 8268
@@
 	-1   0    0    1
 $EndComp
+$Comp
+L MLAB_IO:MICROFC-60035-SMT-TR(1) U2
+U 1 1 5C5D8BBE
+P 9200 2500
+F 0 "U2" H 9022 2553 60  0000 R CNN
+F 1 "MICROFC-60035-SMT-TR(1)" H 9022 2447 60  0000 R CNN
+F 2 "Mlab_IO:MicroFC−60035−SMT" H 9300 2750 60  0001 C CNN
+F 3 "" H 9300 2750 60  0001 C CNN
+	1    9200 2500
+	1    0    0    -1
+$EndComp
+Wire Wire Line
+	9200 2200 9200 2100
+Text Label 9200 2100 0    60   ~ 0
+A
+Text Label 9200 2800 0    60   ~ 0
+K
+$Comp
+L MLAB_IO:MICROFC-60035-SMT-TR(1) U3
+U 1 1 5C5DBA92
+P 10150 2750
+F 0 "U3" H 9972 2803 60  0000 R CNN
+F 1 "MICROFC-60035-SMT-TR(1)" H 9972 2697 60  0000 R CNN
+F 2 "Mlab_IO:MicroFC−60035−SMT" H 10250 3000 60  0001 C CNN
+F 3 "" H 10250 3000 60  0001 C CNN
+	1    10150 2750
+	1    0    0    -1
+$EndComp
+Wire Wire Line
+	9200 2100 10150 2100
+Wire Wire Line
+	10150 2100 10150 2450
+Wire Wire Line
+	9200 2800 9900 2800
+Wire Wire Line
+	9900 2800 9900 3050
+Wire Wire Line
+	9900 3050 10150 3050
 $EndSCHEMATC

Commit message: edit
Parts:
- removed C10, C4, C7: 1u5/50V - NFM41PC155B1H3L, Mlab_L:FIR_1806, symbol Device:EMI_Filter_C
- removed C5, C6: CP, Mlab_C:TantalC_SizeC_Reflow, symbol Device:CP
- removed J1, J2, J3, J4, J7: HEADER_1x01, Mlab_Pin_Headers:Straight_1x01, symbol MLAB_HEADER:HEADER_1x01
- removed J5, J6: CONN_2, Mlab_Pin_Headers:SMD_1_2_4x2, symbol MLAB_Jumpers:CONN_2
- removed U1: ARRAYC-60035-4P-BGA, Mlab_D:ArrayC-60035-4P-BGA, symbol MLAB_IO:ARRAYC-60035-4P-BGA
- removed U3: MICROFC-60035-SMT-TR(1), Mlab_IO:MicroFC−60035−SMT, symbol MLAB_IO:MICROFC-60035-SMT-TR(1)
- added C10: -, symbol Device:C
- added C4, C7: 10u, symbol Device:C
- added C5, C8: 100nF, symbol Device:C
- added C6, C9: 10nF, symbol Device:C
- added D1: M4, symbol Device:D
- added J1, J2, J3, J4, J5, J6, J7, J8: HEADER_2x01_PARALLEL, symbol MLAB_HEADER:HEADER_2x01_PARALLEL
- added R1, R10, R12, R9: 1k, symbol Device:R
- added R11, R5, R6: 0R, symbol Device:R
- added R2, R4: 10R, symbol Device:R
- added R3: 100R, symbol Device:R
- added R7, R8: 2k, symbol Device:R
- added U2: OPA836IDB, Package_TO_SOT_SMD:SOT-23-6, symbol Amplifier_Operational:OPA847xDBV
- C1: renamed from C2; value CP -> 15uF/35V
- C3: value CP -> 47uF
- renumbered C1 to C2, U2 to U1
Connections:
- net labels added: #PD, +28V, +3.3V, +3V6, DIRECT_OUT, OUT
- net labels removed: +, A, K, U1, U1in, U2, U2in, U3, U3in, U4, U4in
- wire segments 61 -> 85
Other:
- note added: "FAST VERSION IN THE SCHEMA"
- note added: "SLOW-RAIL VERSION:\nR6,R7,R8 -\nC10 0R\nR5 10R\n\n"
- moved on the sheet: C1, C2, U1

Commit message: edit
Parts:
- C10, C4, C5, C6, C7, C8, C9, R1, R10, R11, R12, R2, R3, R4, R5, R6, R7, R8, R9: footprint (none) -> Mlab_R:SMD-0805
- D1: footprint (none) -> Mlab_D:Diode-SMA_Standard
- J1, J2, J3, J4, J5, J6, J7, J8: footprint (none) -> Mlab_Pin_Headers:Straight_2x01
Changed lines of the file:
@@
 F 0 "R1" V 2950 2650 50  0000 C CNN
 F 1 "1k" V 3050 2700 50  0000 C CNN
-F 2 "" V 2980 2700 50  0001 C CNN
+F 2 "Mlab_R:SMD-0805" V 2980 2700 50  0001 C CNN
 F 3 "~" H 3050 2700 50  0001 C CNN
 	1    3050 2700
@@
 F 0 "R2" V 3950 2650 50  0000 C CNN
 F 1 "10R" V 4050 2700 50  0000 C CNN
-F 2 "" V 3980 2700 50  0001 C CNN
+F 2 "Mlab_R:SMD-0805" V 3980 2700 50  0001 C CNN
 F 3 "~" H 4050 2700 50  0001 C CNN
 	1    4050 2700
@@
 F 0 "C5" H 4415 2996 50  0000 L CNN
 F 1 "100nF" H 4415 2905 50  0000 L CNN
-F 2 "" H 4338 2800 50  0001 C CNN
+F 2 "Mlab_R:SMD-0805" H 4338 2800 50  0001 C CNN
 F 3 "~" H 4300 2950 50  0001 C CNN
 	1    4300 2950
@@
 F 0 "R4" V 4450 2650 50  0000 C CNN
 F 1 "10R" V 4550 2700 50  0000 C CNN
-F 2 "" V 4480 2700 50  0001 C CNN
+F 2 "Mlab_R:SMD-0805" V 4480 2700 50  0001 C CNN
 F 3 "~" H 4550 2700 50  0001 C CNN
 	1    4550 2700
@@
 F 0 "C6" H 4965 2996 50  0000 L CNN
 F 1 "10nF" H 4965 2905 50  0000 L CNN
-F 2 "" H 4888 2800 50  0001 C CNN
+F 2 "Mlab_R:SMD-0805" H 4888 2800 50  0001 C CNN
 F 3 "~" H 4850 2950 50  0001 C CNN
 	1    4850 2950
@@
 F 0 "C9" H 5415 2996 50  0000 L CNN
 F 1 "10nF" H 5415 2905 50  0000 L CNN
-F 2 "" H 5338 2800 50  0001 C CNN
+F 2 "Mlab_R:SMD-0805" H 5338 2800 50  0001 C CNN
 F 3 "~" H 5300 2950 50  0001 C CNN
 	1    5300 2950
@@
 F 0 "R5" V 6000 4000 50  0000 C CNN
 F 1 "0R" V 6100 4050 50  0000 C CNN
-F 2 "" V 6030 4050 50  0001 C CNN
+F 2 "Mlab_R:SMD-0805" V 6030 4050 50  0001 C CNN
 F 3 "~" H 6100 4050 50  0001 C CNN
 	1    6100 4050
@@
 F 0 "R6" V 6700 3150 50  0000 C CNN
 F 1 "0R" V 6800 3200 50  0000 C CNN
-F 2 "" V 6730 3200 50  0001 C CNN
+F 2 "Mlab_R:SMD-0805" V 6730 3200 50  0001 C CNN
 F 3 "~" H 6800 3200 50  0001 C CNN
 	1    6800 3200
@@
 F 0 "R7" V 7150 2900 50  0000 C CNN
 F 1 "2k" V 7250 2950 50  0000 C CNN
-F 2 "" V 7180 2950 50  0001 C CNN
+F 2 "Mlab_R:SMD-0805" V 7180 2950 50  0001 C CNN
 F 3 "~" H 7250 2950 50  0001 C CNN
 	1    7250 2950
@@
 F 0 "R8" V 7150 4000 50  0000 C CNN
 F 1 "2k" V 7250 4050 50  0000 C CNN
-F 2 "" V 7180 4050 50  0001 C CNN
+F 2 "Mlab_R:SMD-0805" V 7180 4050 50  0001 C CNN
 F 3 "~" H 7250 4050 50  0001 C CNN
 	1    7250 4050
@@
 F 0 "C10" V 6548 3750 50  0000 C CNN
 F 1 "-" V 6639 3750 50  0000 C CNN
-F 2 "" H 6838 3600 50  0001 C CNN
+F 2 "Mlab_R:SMD-0805" H 6838 3600 50  0001 C CNN
 F 3 "~" H 6800 3750 50  0001 C CNN
 	1    6800 3750
@@
 F 0 "R9" V 7600 4700 50  0000 C CNN
 F 1 "1k" V 7700 4750 50  0000 C CNN
-F 2 "" V 7630 4750 50  0001 C CNN
+F 2 "Mlab_R:SMD-0805" V 7630 4750 50  0001 C CNN
 F 3 "~" H 7700 4750 50  0001 C CNN
 	1    7700 4750
@@
 F 0 "R11" V 8200 4100 50  0000 C CNN
 F 1 "0R" V 8300 4150 50  0000 C CNN
-F 2 "" V 8230 4150 50  0001 C CNN
+F 2 "Mlab_R:SMD-0805" V 8230 4150 50  0001 C CNN
 F 3 "~" H 8300 4150 50  0001 C CNN
 	1    8300 4150
@@
 F 0 "R10" V 7900 4500 50  0000 C CNN
 F 1 "1k" V 8000 4550 50  0000 C CNN
-F 2 "" V 7930 4550 50  0001 C CNN
+F 2 "Mlab_R:SMD-0805" V 7930 4550 50  0001 C CNN
 F 3 "~" H 8000 4550 50  0001 C CNN
 	1    8000 4550
@@
 F 0 "R12" V 8750 3800 50  0000 C CNN
 F 1 "1k" V 8850 3850 50  0000 C CNN
-F 2 "" V 8780 3850 50  0001 C CNN
+F 2 "Mlab_R:SMD-0805" V 8780 3850 50  0001 C CNN
 F 3 "~" H 8850 3850 50  0001 C CNN
 	1    8850 3850
@@
 F 0 "C4" H 4165 6196 50  0000 L CNN
 F 1 "10u" H 4165 6105 50  0000 L CNN
-F 2 "" H 4088 6000 50  0001 C CNN
+F 2 "Mlab_R:SMD-0805" H 4088 6000 50  0001 C CNN
 F 3 "~" H 4050 6150 50  0001 C CNN
 	1    4050 6150
@@
 F 0 "C8" H 5365 6196 50  0000 L CNN
 F 1 "100nF" H 5365 6105 50  0000 L CNN
-F 2 "" H 5288 6000 50  0001 C CNN
+F 2 "Mlab_R:SMD-0805" H 5288 6000 50  0001 C CNN
 F 3 "~" H 5250 6150 50  0001 C CNN
 	1    5250 6150
@@
 F 0 "C7" H 4965 6196 50  0000 L CNN
 F 1 "10u" H 4965 6105 50  0000 L CNN
-F 2 "" H 4888 6000 50  0001 C CNN
+F 2 "Mlab_R:SMD-0805" H 4888 6000 50  0001 C CNN
 F 3 "~" H 4850 6150 50  0001 C CNN
 	1    4850 6150
@@
 F 0 "R3" V 4400 5900 50  0000 C CNN
 F 1 "100R" V 4500 5950 50  0000 C CNN
-F 2 "" V 4430 5950 50  0001 C CNN
+F 2 "Mlab_R:SMD-0805" V 4430 5950 50  0001 C CNN
 F 3 "~" H 4500 5950 50  0001 C CNN
 	1    4500 5950
@@
 F 0 "J7" H 9600 3850 60  0000 C CNN
 F 1 "HEADER_2x01_PARALLEL" H 9318 3991 60  0001 C CNN
-F 2 "" H 9400 3850 60  0000 C CNN
+F 2 "Mlab_Pin_Headers:Straight_2x01" H 9400 3850 60  0001 C CNN
 F 3 "" H 9400 3850 60  0000 C CNN
 	1    9400 3850
@@
 F 0 "J8" H 9600 4300 60  0000 C CNN
 F 1 "HEADER_2x01_PARALLEL" H 9318 4441 60  0001 C CNN
-F 2 "" H 9400 4300 60  0000 C CNN
+F 2 "Mlab_Pin_Headers:Straight_2x01" H 9400 4300 60  0001 C CNN
 F 3 "" H 9400 4300 60  0000 C CNN
 	1    9400 4300
@@
 F 0 "J6" H 7950 3100 60  0000 C CNN
 F 1 "HEADER_2x01_PARALLEL" H 7668 3241 60  0001 C CNN
-F 2 "" H 7750 3100 60  0000 C CNN
+F 2 "Mlab_Pin_Headers:Straight_2x01" H 7750 3100 60  0001 C CNN
 F 3 "" H 7750 3100 60  0000 C CNN
 	1    7750 3100
@@
 F 0 "D1" V 3154 6229 50  0000 L CNN
 F 1 "M4" V 3245 6229 50  0000 L CNN
-F 2 "" H 3200 6150 50  0001 C CNN
+F 2 "Mlab_D:Diode-SMA_Standard" H 3200 6150 50  0001 C CNN
 F 3 "~" H 3200 6150 50  0001 C CNN
 	1    3200 6150
@@
 F 0 "J4" H 2800 5800 60  0000 C CNN
 F 1 "HEADER_2x01_PARALLEL" H 2518 5941 60  0001 C CNN
-F 2 "" H 2600 5800 60  0000 C CNN
+F 2 "Mlab_Pin_Headers:Straight_2x01" H 2600 5800 60  0001 C CNN
 F 3 "" H 2600 5800 60  0000 C CNN
 	1    2600 5800
@@
 F 0 "J5" H 2800 5900 60  0000 C CNN
 F 1 "HEADER_2x01_PARALLEL" H 2518 6041 60  0001 C CNN
-F 2 "" H 2600 5900 60  0000 C CNN
+F 2 "Mlab_Pin_Headers:Straight_2x01" H 2600 5900 60  0001 C CNN
 F 3 "" H 2600 5900 60  0000 C CNN
 	1    2600 5900
@@
 F 0 "J2" H 2700 2700 60  0000 C CNN
 F 1 "HEADER_2x01_PARALLEL" H 2418 2841 60  0001 C CNN
-F 2 "" H 2500 2700 60  0000 C CNN
+F 2 "Mlab_Pin_Headers:Straight_2x01" H 2500 2700 60  0001 C CNN
 F 3 "" H 2500 2700 60  0000 C CNN
 	1    2500 2700
@@
 F 0 "J3" H 2700 2800 60  0000 C CNN
 F 1 "HEADER_2x01_PARALLEL" H 2418 2941 60  0001 C CNN
-F 2 "" H 2500 2800 60  0000 C CNN
+F 2 "Mlab_Pin_Headers:Straight_2x01" H 2500 2800 60  0001 C CNN
 F 3 "" H 2500 2800 60  0000 C CNN
 	1    2500 2800
@@
 F 0 "J1" H 2700 2600 60  0000 C CNN
 F 1 "HEADER_2x01_PARALLEL" H 2418 2741 60  0001 C CNN
-F 2 "" H 2500 2600 60  0000 C CNN
+F 2 "Mlab_Pin_Headers:Straight_2x01" H 2500 2600 60  0001 C CNN
 F 3 "" H 2500 2600 60  0000 C CNN
 	1    2500 2600

Commit message: edit
Parts:
- added J4, J9: HEADER_2x01_PARALLEL, Mlab_Pin_Headers:Straight_2x01, symbol MLAB_HEADER:HEADER_2x01_PARALLEL
- renumbered J8 to J10, J4 to J5, J5 to J6, J6 to J7, J7 to J8
Connections:
- net GND: now also J4.1, J4.2, J9.1, J9.2
Changed lines of the file:
@@
-$EndComp
-$Comp
-L MLAB_MECHANICAL:HOLE M2
-U 1 1 549D7628
-P 10400 700
-F 0 "M2" V 10300 700 60  0000 C CNN
-F 1 "HOLE" H 10400 600 60  0001 C CNN
-F 2 "Mlab_Mechanical:MountingHole_3mm" H 10400 700 60  0001 C CNN
-F 3 "" H 10400 700 60  0000 C CNN
-	1    10400 700
-	0    -1   -1   0
-$EndComp
-$Comp
-L MLAB_MECHANICAL:HOLE M3
-U 1 1 549D7646
-P 10600 700
-F 0 "M3" V 10500 700 60  0000 C CNN
-F 1 "HOLE" H 10600 600 60  0001 C CNN
-F 2 "Mlab_Mechanical:MountingHole_3mm" H 10600 700 60  0001 C CNN
-F 3 "" H 10600 700 60  0000 C CNN
-	1    10600 700
-	0    -1   -1   0
 $EndComp
 $Comp
@@
 $EndComp
 Wire Notes Line
-	10100 550  11100 550
-Wire Notes Line
 	11100 550  11100 950
-Wire Notes Line
-	11100 950  10100 950
-Wire Notes Line
-	10100 950  10100 550
 Text Notes 10100 950  0    60   ~ 0
 MOUNTING HOLES
 $Comp
-L power:GND #PWR022
+L power:GND #PWR023
 U 1 1 5BAC7DDD
 P 11000 650
-F 0 "#PWR022" H 11000 400 50  0001 C CNN
+F 0 "#PWR023" H 11000 400 50  0001 C CNN
 F 1 "GND" H 11005 477 50  0000 C CNN
 F 2 "" H 11000 650 50  0001 C CNN
@@
 +3V6
 $Comp
-L MLAB_HEADER:HEADER_2x01_PARALLEL J7
+L MLAB_HEADER:HEADER_2x01_PARALLEL J8
 U 1 1 5C73FBA4
 P 9400 3850
-F 0 "J7" H 9600 3850 60  0000 C CNN
+F 0 "J8" H 9600 3850 60  0000 C CNN
 F 1 "HEADER_2x01_PARALLEL" H 9318 3991 60  0001 C CNN
 F 2 "Mlab_Pin_Headers:Straight_2x01" H 9400 3850 60  0001 C CNN
@@
 $EndComp
 $Comp
-L MLAB_HEADER:HEADER_2x01_PARALLEL J8
+L MLAB_HEADER:HEADER_2x01_PARALLEL J10
 U 1 1 5C73FDF3
 P 9400 4300
-F 0 "J8" H 9600 4300 60  0000 C CNN
+F 0 "J10" H 9600 4300 60  0000 C CNN
 F 1 "HEADER_2x01_PARALLEL" H 9318 4441 60  0001 C CNN
 F 2 "Mlab_Pin_Headers:Straight_2x01" H 9400 4300 60  0001 C CNN
@@
 $EndComp
 $Comp
-L MLAB_HEADER:HEADER_2x01_PARALLEL J6
+L MLAB_HEADER:HEADER_2x01_PARALLEL J7
 U 1 1 5C73FF81
 P 7750 3100
-F 0 "J6" H 7950 3100 60  0000 C CNN
+F 0 "J7" H 7950 3100 60  0000 C CNN
 F 1 "HEADER_2x01_PARALLEL" H 7668 3241 60  0001 C CNN
 F 2 "Mlab_Pin_Headers:Straight_2x01" H 7750 3100 60  0001 C CNN
@@
 Connection ~ 3200 5950
 $Comp
-L MLAB_HEADER:HEADER_2x01_PARALLEL J4
+L MLAB_HEADER:HEADER_2x01_PARALLEL J5
 U 1 1 5C749873
 P 2600 5800
-F 0 "J4" H 2800 5800 60  0000 C CNN
+F 0 "J5" H 2800 5800 60  0000 C CNN
 F 1 "HEADER_2x01_PARALLEL" H 2518 5941 60  0001 C CNN
 F 2 "Mlab_Pin_Headers:Straight_2x01" H 2600 5800 60  0001 C CNN
@@
 $EndComp
 $Comp
-L MLAB_HEADER:HEADER_2x01_PARALLEL J5
+L MLAB_HEADER:HEADER_2x01_PARALLEL J6
 U 1 1 5C74D68D
 P 2600 5900
-F 0 "J5" H 2800 5900 60  0000 C CNN
+F 0 "J6" H 2800 5900 60  0000 C CNN
 F 1 "HEADER_2x01_PARALLEL" H 2518 6041 60  0001 C CNN
 F 2 "Mlab_Pin_Headers:Straight_2x01" H 2600 5900 60  0001 C CNN
@@
 Text Notes 9600 2250 0    60   ~ 0
 SLOW-RAIL VERSION:\nR6,R7,R8 -\nC10 0R\nR5 10R\n\n
+$Comp
+L MLAB_MECHANICAL:HOLE M3
+U 1 1 5C6D1820
+P 10600 700
+F 0 "M3" V 10500 700 60  0000 C CNN
+F 1 "HOLE" H 10600 600 60  0001 C CNN
+F 2 "Mlab_Mechanical:MountingHole_3mm" H 10600 700 60  0001 C CNN
+F 3 "" H 10600 700 60  0000 C CNN
+	1    10600 700
+	0    -1   -1   0
+$EndComp
+$Comp
+L MLAB_MECHANICAL:HOLE M2
+U 1 1 5C6D1882
+P 10400 700
+F 0 "M2" V 10300 700 60  0000 C CNN
+F 1 "HOLE" H 10400 600 60  0001 C CNN
+F 2 "Mlab_Mechanical:MountingHole_3mm" H 10400 700 60  0001 C CNN
+F 3 "" H 10400 700 60  0000 C CNN
+	1    10400 700
+	0    -1   -1   0
+$EndComp
+Wire Notes Line
+	9700 550  9700 950
+Wire Notes Line
+	9700 550  11100 550
+Wire Notes Line
+	9700 950  11100 950
+$Comp
+L MLAB_HEADER:HEADER_2x01_PARALLEL J4
+U 1 1 5C6DBC7D
+P 2600 5700
+F 0 "J4" H 2800 5700 60  0000 C CNN
+F 1 "HEADER_2x01_PARALLEL" H 2518 5841 60  0001 C CNN
+F 2 "Mlab_Pin_Headers:Straight_2x01" H 2600 5700 60  0001 C CNN
+F 3 "" H 2600 5700 60  0000 C CNN
+	1    2600 5700
+	-1   0    0    1
+$EndComp
+Wire Wire Line
+	2850 5700 2900 5700
+Wire Wire Line
+	2900 5700 2900 5900
+Connection ~ 2900 5900
+$Comp
+L MLAB_HEADER:HEADER_2x01_PARALLEL J9
+U 1 1 5C6DECB4
+P 9400 3950
+F 0 "J9" H 9600 3950 60  0000 C CNN
+F 1 "HEADER_2x01_PARALLEL" H 9318 4091 60  0001 C CNN
+F 2 "Mlab_Pin_Headers:Straight_2x01" H 9400 3950 60  0001 C CNN
+F 3 "" H 9400 3950 60  0000 C CNN
+	1    9400 3950
+	1    0    0    -1
+$EndComp
+$Comp
+L power:GND #PWR022
+U 1 1 5C6DEE35
+P 9100 4000
+F 0 "#PWR022" H 9100 3750 50  0001 C CNN
+F 1 "GND" H 9105 3827 50  0000 C CNN
+F 2 "" H 9100 4000 50  0001 C CNN
+F 3 "" H 9100 4000 50  0001 C CNN
+	1    9100 4000
+	1    0    0    -1
+$EndComp
+Wire Wire Line
+	9150 3950 9100 3950
+Wire Wire Line
+	9100 3950 9100 4000
 $EndSCHEMATC

Commit message: edit
Parts:
- U2: UST_ID (none) -> 5c7273171287500b4e112ff8
Changed lines of the file:
@@
 EESchema Schematic File Version 4
 LIBS:AIRDOSC01A_PCB01A-cache
-EELAYER 26 0
+EELAYER 29 0
 EELAYER END
 $Descr A4 11693 8268
@@
 F 2 "Package_TO_SOT_SMD:SOT-23-6" H 8100 3850 50  0001 C CNN
 F 3 "http://www.ti.com/lit/ds/symlink/opa847.pdf" H 8100 4050 50  0001 C CNN
+F 4 "5c7273171287500b4e112ff8" H 8100 3850 50  0001 C CNN "UST_ID"
 	1    8100 3850
 	1    0    0    -1
