File: hw/sch_pcb/AIRDOSC01A_PCB01B/hw/sch_pcb/AIRDOSC01A_PCB01B.kicad_pcb (KiCad board)
At the start: 2 copper layers, 30 x 40.1 mm, 39 parts, among them J1 HEADER_2x01_PARALLEL, J10 HEADER_2x01_PARALLEL, J2 HEADER_2x01_PARALLEL, J3 HEADER_2x01_PARALLEL, J4 HEADER_2x01_PARALLEL, J5 HEADER_2x01_PARALLEL, J6 HEADER_2x01_PARALLEL, J7 HEADER_2x01_PARALLEL, J8 HEADER_2x01_PARALLEL, J9 HEADER_2x01_PARALLEL, M1 HOLE, M2 HOLE, M3 HOLE, M4 HOLE, U1 MICROFC-60035-SMT-TR(1), U2 OPA836IDB

Commit message: Úprava hodnot ve schématu.
Parts:
- C10: value - -> 0R
- C6: value 10nF -> 100nF
- R1: value 1k -> 10R
- R10: value 1k -> 6k8
- R11: value 0R -> 1k
- R5: value 0R -> 10R
- R6: value 0R -> -
- R7: value 2k -> -
- R8: value 2k -> 100nF
- R9: value 1k -> 470R
