File: hw/sch_pcb/AIRDOSC01A_PCB01C/hw/sch_pcb/AIRDOSC01A_PCB01C.kicad_pcb (KiCad board)
At the start: 2 copper layers, 30 x 40.1 mm, 39 parts, among them J1 HEADER_2x01_PARALLEL, J10 HEADER_2x01_PARALLEL, J2 HEADER_2x01_PARALLEL, J3 HEADER_2x01_PARALLEL, J4 HEADER_2x01_PARALLEL, J5 HEADER_2x01_PARALLEL, J6 HEADER_2x01_PARALLEL, J7 HEADER_2x01_PARALLEL, J8 HEADER_2x01_PARALLEL, J9 HEADER_2x01_PARALLEL, M1 HOLE, M2 HOLE, M3 HOLE, M4 HOLE, U1 MICROFC-60035-SMT-TR(1), U2 OPA836IDB

Commit message: Change R10 from 6k8 to 12k
Parts:
- R10: value 6k8 -> 12k
Changed lines of the file:
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@@
-(kicad_pcb (version 20210228) (generator pcbnew)
+(kicad_pcb (version 20211014) (generator pcbnew)
   (general
     (thickness 1.6)
@@
     (property "Sheetfile" "AIRDOSC01A_PCB01C.kicad_sch")
     (property "Sheetname" "")
-    (property "UST_ID" "5c70984612875079b91f899a")
+    (property "UST_ID" "5c70984612875079b91f89a1")
     (attr smd)
     (fp_text reference "R10" (at 0 0.3175) (layer "B.Fab")
       (effects (font (size 0.50038 0.50038) (thickness 0.10922)) (justify mirror))
     )
-    (fp_text value "6k8" (at 0.127 -0.381) (layer "B.Fab")
+    (fp_text value "12k" (at 0.127 -0.381) (layer "B.Fab")
       (effects (font (size 0.50038 0.50038) (thickness 0.10922)) (justify mirror))
     )
@@
       (net 14 "Net-(R10-Pad2)") (pinfunction "-") (pintype "input"))
     (pad "5" smd rect locked (at 1.1 0) (size 1.06 0.65) (layers "B.Cu" "B.Paste" "B.Mask")
-      (net 12 "/#PD") (pinfunction "~DIS") (pintype "input"))
+      (net 12 "/#PD") (pinfunction "~{DIS}") (pintype "input"))
     (pad "6" smd rect locked (at 1.1 0.95) (size 1.06 0.65) (layers "B.Cu" "B.Paste" "B.Mask")
       (net 7 "+3V3") (pinfunction "V+") (pintype "power_in"))
@@
     )
   )
-  (gr_poly (pts
- (xy 24.384 -40.132)
-    (xy 24.384 -0.508)
-    (xy 29.972 -0.508)
-    (xy 29.972 -40.132)) (layer "F.Mask") (width 0.15) (fill solid))
+  (gr_poly
+    (pts
+      (xy 24.384 -40.132)
+      (xy 24.384 -0.508)
+      (xy 29.972 -0.508)
+      (xy 29.972 -40.132)
+    ) (layer "F.Mask") (width 0.15) (fill solid))
   (gr_line (start 30.353 -0.254) (end 30.353 -40.386) (layer "Edge.Cuts") (width 0.15))
   (gr_line (start 0.381 -0.254) (end 0.381 -40.386) (layer "Edge.Cuts") (width 0.15))
